File: EagleCad/PCM3060 Guitar Cape/PCM3060 Guitar Cape.brd (EAGLE design)
At the start: 86.4 x 54.6 mm, 50 parts, among them J1 MONOSW, J2 MONOSW, U2 PCM3060_PW_28, U3 LM386

Commit message: Fixed Grounding Issue on Output Jack
Previously, the switched 1/4" output jack for the system would be
grounded when no cable was connected. This is correct for the input,
however grounding the output of the system is not proper.
Connections:
- net GND: no longer J2.TN
Changed lines of the file:
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@@
 <contactref element="R22" pad="2"/>
 <contactref element="C20" pad="2"/>
-<contactref element="J2" pad="TN"/>
 <contactref element="J2" pad="SN"/>
 <contactref element="J2" pad="S"/>
